Commit message: modified urdf

File: src/robot_arm_description/urdf/robot_arm.urdf (robot description, URDF)
Before this commit: robot robot_arm, 6 links, 5 joints
Links:
- removed link link2
- removed link link3
- removed link link4
- removed link link5
- added link link_1, mass 1.0444299778861974; collision mesh filename=file:///home/wwd9861/robot_arm_ws/src/robot_arm_description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 scale=0.001 0.001 0.001; visual mesh filename=file:///home/wwd9861/robot_arm_ws/src/robot_arm_description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 scale=0.001 0.001 0.001
- added link link_2, mass 1.0723019224070054; collision mesh filename=file:///home/wwd9861/robot_arm_ws/src/robot_arm_description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 scale=0.001 0.001 0.001; visual mesh filename=file:///home/wwd9861/robot_arm_ws/src/robot_arm_description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 scale=0.001 0.001 0.001
- added link link_3, mass 1.0723019224070065; collision mesh filename=file:///home/wwd9861/robot_arm_ws/src/robot_arm_description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 scale=0.001 0.001 0.001; visual mesh filename=file:///home/wwd9861/robot_arm_ws/src/robot_arm_description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 scale=0.001 0.001 0.001
- added link link_4, mass 0.28036972878940647; collision mesh filename=file:///home/wwd9861/robot_arm_ws/src/robot_arm_description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 scale=0.001 0.001 0.001; visual mesh filename=file:///home/wwd9861/robot_arm_ws/src/robot_arm_description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 scale=0.001 0.001 0.001
- link base_link: mass 0.5 -> 2.1649980446638213
Joints:
- joint revolute1: child link2 -> link_1; limit lower=-1.570796 upper=1.570796 effort=10 velocity=20.0 -> lower=-3.141592 upper=3.141592 effort=10 velocity=20.0; origin xyz=0.0 0.0425 0.053 rpy=0 0 0 -> xyz=0.022 0.0 0.0638 rpy=0 0 0
- joint revolute2: axis 1.0 0.0 0.0 -> 1.0 0.0 -0.0; child link3 -> link_2; origin xyz=-0.024625 0.0 0.063 rpy=0 0 0 -> xyz=-0.025 0.0002 0.054 rpy=0 0 0; parent link2 -> link_1
- joint revolute3: axis -1.0 -0.0 -0.0 -> 1.0 -0.0 0.0; child link4 -> link_3; limit lower=0.0 upper=3.141592 effort=10 velocity=20.0 -> lower=-3.141592 upper=0.0 effort=10 velocity=20.0; origin xyz=0.0 0.0 0.105 rpy=0 0 0 -> xyz=0.0 0.0002 0.105 rpy=0 0 0; parent link3 -> link_2
- joint revolute4: axis 1.0 -0.0 0.0 -> 1.0 0.0 0.0; child link5 -> link_4; origin xyz=0.0 0.0 0.105 rpy=0 0 0 -> xyz=0.0 -0.0002 0.105 rpy=0 0 0; parent link4 -> link_3

Commit message: modified

File: src/robot_arm_description/urdf/robot_arm.urdf (robot description, URDF)
Before this commit: robot robot_arm, 6 links, 5 joints
Joints:
- joint revolute1: origin xyz=0.022 0.0 0.0638 rpy=0 0 0 -> xyz=0.0 0.0 0.062 rpy=0 0 0

Commit message: update

File: src/robot_arm_description/urdf/robot_arm.urdf (robot description, URDF)
Before this commit: robot robot_arm, 6 links, 5 joints
Links:
- added link rotate, mass 0.6631591419630531; collision mesh filename=file:///home/wwd9861/robot_arm_ws/src/robot_arm_description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 scale=0.001 0.001 0.001; visual mesh filename=file:///home/wwd9861/robot_arm_ws/src/robot_arm_description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 scale=0.001 0.001 0.001
- link base_link: mass 2.1649980446638213 -> 2.5305930297877364
- link link_1: mass 1.0444299778861974 -> 0.7144960689551971
- link link_2: mass 1.0723019224070054 -> 1.0723019224070052
Joints:
- added joint fixed1: type fixed, parent rotate, child link_1, origin xyz=-0.0 0.0 0.01 rpy=0 0 0
- joint revolute1: child link_1 -> rotate; origin xyz=0.0 0.0 0.062 rpy=0 0 0 -> xyz=0.0 0.0 0.1116 rpy=0 0 0
- joint revolute2: axis 1.0 0.0 -0.0 -> -1.0 0.0 0.0; limit lower=-1.570796 upper=1.570796 effort=10 velocity=20.0 -> lower=-3.141592 upper=3.141592 effort=10 velocity=20.0; origin xyz=-0.025 0.0002 0.054 rpy=0 0 0 -> xyz=-0.025 0.0 0.045 rpy=0 0 0
- joint revolute3: axis 1.0 -0.0 0.0 -> -1.0 -0.0 0.0; limit lower=-3.141592 upper=0.0 effort=10 velocity=20.0 -> lower=-3.141592 upper=3.141592 effort=10 velocity=20.0
- joint revolute4: axis 1.0 0.0 0.0 -> -1.0 0.0 0.0; limit lower=-1.570796 upper=1.570796 effort=10 velocity=20.0 -> lower=-3.141592 upper=3.141592 effort=10 velocity=20.0
